File: Dronev1 STM32/Dronev1.kicad_pcb (KiCad board)
At the start: 2 copper layers, 70 x 70 mm, 36 parts, among them J7 JST_2mm_LiPo, J8 USB3131-30-0230-A_REVB, Q1 PMOS, SW1 SMD_6.2x6.2mm_h7.0mm, SW2 SMD_6.2x6.2mm_h7.0mm, U1 STM32F415RGTx, U2 MIC5219-3.3YM5, U3 LSM6DS3, U4 ESP8266EX

Commit message: PCB complete, needs branding and attention to a few warnings but not critical
Parts:
- removed Q1: PMOS, PMOS_DMP2066UFDE-7:MOSFET_DMP2066UFDE-7
- added Q2: PMOS_DGS, SparkFun-Semiconductor-Standard:SOT23-3, F.Cu at (185.5, 112.4)
- moved C2 57.6 mm to (158.5, 132.0), turned to 180 degrees
- moved R7 46.1 mm to (141.0, 129.5)
- moved R9 42.2 mm to (145.5, 116.0), turned to 0 degrees
- moved R8 42.1 mm to (141.0, 127.5)
- moved C6 32.6 mm to (140.0, 107.5)
- moved R3 18.0 mm to (141.0, 133.5)
- moved D2 10.9 mm to (171.0, 122.5)
- moved R1 7.62 mm to (159.5, 126.5)
- moved U1 5.02 mm to (153.0, 110.0)
- moved C7 3.04 mm to (183.5, 90.0), turned to 0 degrees
- moved C4 3.04 mm to (146.0, 77.0)
- moved USB_J2 2.06 mm to (134.0, 140.0)
- moved U4 1.58 mm to (149.5, 94.0), turned to 90 degrees
- moved J1 1.50 mm to (181.0, 138.0)
- turned D1 to 180 degrees
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- renumbered C7 to C1, C5 to C10, C9 to C2, C6 to C3, C10 to C4, C1 to C5, C4 to C6, C2 to C7, C3 to C8, C8 to C9, D2 to D1, D4 to D2, ESC2 to ESC1, ESC1 to ESC2, J7 to J1, R6 to R1, R1 to R10, R5 to R2, R4 to R3, R7 to R4, R2 to R5, R3 to R6, R11 to R7, R12 to R8, R8 to R9, SW2 to SW1, SW1 to SW2, U3 to U1, U4 to U3, U1 to U4, J8 to USB_J2
Connections:
- U4 pad 18: unconnected-(U1-VSS-Pad18) -> /unconnected-(U4-VSS-Pad18)_1
- U4 pad 63: unconnected-(U1-VSS-Pad18)_1 -> /unconnected-(U4-VSS-Pad18)_1_1
- USB_J2 pad S1: unconnected-(J8-SHIELD-PadS1)_1 -> /unconnected-(J2-SHIELD-PadS1)_1_1
- USB_J2 pad S2: unconnected-(J8-SHIELD-PadS1) -> /unconnected-(J2-SHIELD-PadS1)_1
Routing:
- net GND: track 307.4 -> 51.8 mm, vias 15 -> 8
- net /USB_D-: track 8.90 -> 118.6 mm, vias 0 -> 4
- net /USB_D+: track 4.62 -> 104.5 mm, vias 0 -> 4
- net /V_{BATT}: track 142.8 -> 47.7 mm, vias 2 -> 0
- net /USART2_TX: track 119.5 -> 36.5 mm, vias 2 -> 4
- net /USART2_RX: track 116.7 -> 34.0 mm, vias 0 -> 2
- net /SLAVE_SDA: track 51.2 -> 122.6 mm
- net Net-(J2-D+): track 104.3 -> 40.0 mm, vias 1 -> 4
- net Net-(J2-D-): track 73.9 -> 15.2 mm, vias 0 -> 1
- net /SLAVE_INT1: track 67.8 -> 14.5 mm, vias 4 -> 2
- net Net-(Q2-D): track 58.5 -> 16.4 mm, vias 1 -> 0
- net Net-(D2-A): track 20.6 -> 59.8 mm, vias 1 -> 6
- net +3.3V: track 311.0 -> 273.8 mm, vias 16 -> 0
- net Net-(U2-BP): track 50.8 -> 14.2 mm, vias 2 -> 0
- net /SLAVE_SCL: track 71.3 -> 98.3 mm, vias 9 -> 3
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- added copper zone on B.Cu, net GND
- added copper zone on F.Cu, net GND
Other:
- board size 70 x 70 mm -> 70 x 72.5 mm

Commit message: friday the 3rd version
Parts:
- renumbered SW1 to ON/OFF
Changed lines of the file:
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@@
 		(descr "https://www.we-online.com/components/products/datasheet/4301x2xxx8x6.pdf")
 		(tags "SparkFun Momentary Switch (Pushbutton)")
-		(property "Reference" "SW1"
-			(at 0 -3.175 90)
+		(property "Reference" "ON/OFF"
+			(at 0 5 90)
 			(layer "F.Fab")
 			(effects
 				(font
-					(size 0.5 0.5)
-					(thickness 0.1)
+					(size 0.8 0.5)
+					(thickness 0.098425)
+					(bold yes)
 				)
 				(justify bottom)
